File: kicad/mcu_board/mcu_board.kicad_pcb (KiCad board)
At the start: 2 copper layers, 30 parts, among them J1 Buttons, J10 Lights, J2 Humidity, J3 IR, J4 Power Monitor, J5 Photoresistor, J6 24V In, J7 5V Out, J8 Programmer, J9 Power Board, SW1 Reset, U1 ATmega328-P, X1 CXO_DIP8

Commit message: finished up MCU board
Parts:
- removed J10: Lights, Connector_PinHeader_2.54mm:PinHeader_1x04_P2.54mm_Vertical
- removed X1: CXO_DIP8, Oscillator:Oscillator_DIP-8
- added Crystal: 16MHz, Crystal:Crystal_HC49-U_Vertical, F.Cu at (121.0, 116.0)
- added D1: SBR80520, Diode_SMD:D_SOD-123, F.Cu at (128.3, 91.6)
- added Lights: Lights, Connector_PinHeader_2.54mm:PinHeader_1x04_P2.54mm_Vertical, F.Cu at (131.8, 129.9)
- C1, C4, C6, C7, C8, C9: footprint Capacitor_SMD:C_0201_0603Metric_Pad0.64x0.40mm_HandSolder -> Capacitor_SMD:C_0603_1608Metric_Pad1.08x0.95mm_HandSolder
- moved H1 76.2 mm to (98.7, 78.1)
- moved 24V 66.8 mm to (101.0, 84.8), turned to -90 degrees
- moved H2 52.6 mm to (98.7, 135.1)
- moved Humidity 45.9 mm to (146.9, 84.7), turned to -90 degrees
- moved Sol 42.6 mm to (129.9, 84.7), turned to 90 degrees
- moved C4 40.3 mm to (128.5, 109.6), turned to -90 degrees
- moved ISP 39.7 mm to (120.0, 86.6), turned to -90 degrees
- moved C11 38.8 mm to (110.9, 100.6), turned to -90 degrees
- moved Photo. 38.6 mm to (144.0, 118.7), turned to 180 degrees
- moved Reset 37.0 mm to (117.3, 100.6)
- moved H3 36.5 mm to (150.7, 78.1)
- moved R6 35.7 mm to (125.1, 100.6), turned to 90 degrees
- moved Out 33.5 mm to (100.0, 119.8), turned to 90 degrees
- moved C2 33.3 mm to (109.9, 108.5), turned to -90 degrees
- moved J1 33.1 mm to (127.1, 123.3)
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- renumbered J6 to 24V, PS1 to DC-DC, J2 to Humidity, J3 to IR, J8 to ISP, U1 to MCU, J4 to Monitor, J7 to Out, J5 to Photo., SW1 to Reset, J9 to Sol
Connections:
- C10 pad 1: GND1 -> MCU_XTAL1
- C10 pad 2: MCU_XTAL1 -> GND1
- ISP pad 2: +5V -> Net-(J8-Pad2)
Routing:
- net +5V: track 0.00 -> 127.5 mm
- net MCU_N_RESET: track 0.00 -> 54.4 mm
- net MCU_MOSI: track 0.00 -> 42.7 mm, vias 0 -> 2
- net MCU_MISO: track 0.00 -> 41.4 mm, vias 0 -> 2
- net MCU_SCK: track 0.00 -> 38.8 mm, vias 0 -> 2
- net Resistor: track 0.00 -> 23.1 mm
- net Grid: track 0.00 -> 20.7 mm
- net Solar: track 0.00 -> 18.4 mm
- net MCU_XTAL1: track 0.00 -> 18.1 mm
- net SDA: track 0.00 -> 17.8 mm
- net MCU_XTAL2: track 0.00 -> 17.1 mm
- net Photoresistor: track 0.00 -> 14.7 mm
- net SCL: track 0.00 -> 14.0 mm
- net Red: track 0.00 -> 12.5 mm
- net +24V: track 0.00 -> 11.9 mm
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- added copper zone on B.Cu, net GND1
- added copper zone on F.Cu, net GND1
Other:
- board outline added: 59.6 x 64.4 mm
- board text added: "+"
- board text added: "-"
- board text added: "5V"
- board text added: "5V Out"
- board text added: "G"
- board text added: "Grid"
- board text added: "MOSFETs"
- board text added: "Photo. In"
- board text added: "R"
- board text added: "SCL"
- board text added: "SDA"
- board text added: "Team 20 MCU Board v1 3/7/22"
- board text added: "Vo"
- board text added: "W"
- board text added: "Y"

Commit message: finishing up MCU and adding gerbers
Parts:
- removed 24V: 24V In, Connector_PinHeader_2.54mm:PinHeader_1x02_P2.54mm_Vertical
- removed C4, C7, C9: 0.1uF, Capacitor_SMD:C_0603_1608Metric_Pad1.08x0.95mm_HandSolder
- removed Crystal: 16MHz, Crystal:Crystal_HC49-U_Vertical
- removed DC-DC: SPBW03F-05, SamacSys_Parts:SPBW06F05
- removed Humidity: Humidity, Connector_PinHeader_2.54mm:PinHeader_1x04_P2.54mm_Vertical
- removed IR: IR, Connector_PinHeader_2.54mm:PinHeader_1x03_P2.54mm_Vertical
- removed ISP: Programmer, Connector_IDC:IDC-Header_2x03_P2.54mm_Vertical
- removed Lights: Lights, Connector_PinHeader_2.54mm:PinHeader_1x04_P2.54mm_Vertical
- removed MCU: ATmega328-P, Package_DIP:DIP-28_W7.62mm
- removed Monitor: Power Monitor, Connector_PinHeader_2.54mm:PinHeader_1x02_P2.54mm_Vertical
- removed Out: 5V Out, Connector_PinHeader_2.54mm:PinHeader_1x03_P2.54mm_Vertical
- removed Photo.: Photoresistor, Connector_PinHeader_2.54mm:PinHeader_1x02_P2.54mm_Vertical
- removed Reset: Reset, Button_Switch_SMD:SW_SPST_TL3305B
- removed Sol: Power Board, Connector_PinHeader_2.54mm:PinHeader_1x03_P2.54mm_Vertical
- added J10: Lights, Connector_PinHeader_2.54mm:PinHeader_1x04_P2.54mm_Vertical, F.Cu at (230.8, 132.1)
- added J2: Humidity, Connector_PinHeader_2.54mm:PinHeader_1x04_P2.54mm_Vertical, F.Cu at (254.9, 100.6)
- added J3: IR, Connector_PinHeader_2.54mm:PinHeader_1x03_P2.54mm_Vertical, F.Cu at (248.3, 101.7)
- added J4: Power Monitor, Connector_PinHeader_2.54mm:PinHeader_1x02_P2.54mm_Vertical, F.Cu at (241.8, 93.1)
- added J5: Photoresistor, Connector_PinHeader_2.54mm:PinHeader_1x02_P2.54mm_Vertical, F.Cu at (248.4, 109.5)
- added J6: 24V In, Connector_PinHeader_2.54mm:PinHeader_1x02_P2.54mm_Vertical, F.Cu at (195.2, 93.2)
- added J7: 5V Out, Connector_PinHeader_2.54mm:PinHeader_1x03_P2.54mm_Vertical, F.Cu at (194.2, 129.2)
- added J8: Programmer, Connector_IDC:IDC-Header_2x03_P2.54mm_Vertical, F.Cu at (214.8, 95.0)
- added J9: Power Board, Connector_PinHeader_2.54mm:PinHeader_1x03_P2.54mm_Vertical, F.Cu at (222.4, 93.1)
- added PS1: SPBW03F-05, SamacSys_Parts:SPBW06F05, F.Cu at (197.6, 99.8)
- added SW1: Reset, Button_Switch_SMD:SW_SPST_TL3305B, F.Cu at (212.3, 107.3)
- added U1: ATmega328-P, Package_DIP:DIP-28_W7.62mm, F.Cu at (230.8, 92.8)
- added Y1: 16MHz, Crystal:Crystal_HC49-U_Vertical, F.Cu at (224.3, 112.6)
- moved C8 119.3 mm to (241.7, 113.2), turned to 0 degrees
- moved C10 112.5 mm to (228.3, 112.0), turned to 90 degrees
- moved C12 112.5 mm to (228.3, 116.5), turned to -90 degrees
- moved C11 107.5 mm to (218.2, 107.3)
- moved H3 106.3 mm to (256.8, 86.1)
- moved H4 106.3 mm to (256.8, 141.9)
- moved C6 101.0 mm to (227.5, 106.5), turned to 180 degrees
- moved C1 99.1 mm to (241.7, 110.6)
- moved J1 96.7 mm to (223.6, 129.5)
- moved R1 95.8 mm to (241.7, 106.9), turned to -90 degrees
- moved D1 95.2 mm to (223.1, 98.9)
- moved H1 95.0 mm to (193.3, 86.1)
- moved H2 94.9 mm to (193.3, 141.9)
- moved C2 94.4 mm to (204.1, 113.8)
- moved R6 81.6 mm to (206.4, 107.4)
Routing:
- net +5V: track 127.5 -> 217.6 mm
- net MCU_MOSI: track 42.7 -> 58.9 mm, vias 2 -> 0
- net MCU_SCK: track 38.8 -> 53.5 mm, vias 2 -> 0
- net GND1: track 6.15 -> 19.5 mm, vias 6 -> 9
- net MCU_MISO: track 41.4 -> 53.7 mm, vias 2 -> 0
- net MCU_XTAL1: track 18.1 -> 6.70 mm
- net MCU_XTAL2: track 17.1 -> 7.33 mm
- net Solar: track 18.4 -> 9.64 mm
- net Grid: track 20.7 -> 12.8 mm
- net Resistor: track 23.1 -> 15.9 mm
- net Bike: track 4.80 -> 11.0 mm
- net Vo: track 5.52 -> 11.5 mm
- net Pedestrian: track 4.80 -> 10.6 mm
- net Photoresistor: track 14.7 -> 10.6 mm
- net MCU_N_RESET: track 54.4 -> 57.8 mm, vias 0 -> 4
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- removed copper zone on F.Cu, net GND1
Other:
- board size 59.6 x 64.4 mm -> 71 x 62.9 mm
- board text removed: "+"
- board text removed: "-"
- board text removed: "5V"
- board text removed: "5V Out"
- board text removed: "G"
- board text removed: "Grid"
- board text removed: "MOSFETs"
- board text removed: "Photo. In"
- board text removed: "R"
- board text removed: "SCL"
- board text removed: "SDA"
- board text removed: "Vo"
- board text removed: "W"
- board text removed: "Y"
