File: kicad/light_board/light_board.kicad_pcb (KiCad board)
At the start: 2 copper layers, 85 x 50 mm, 35 parts, among them J1 24V, J10 Screw_Terminal_01x02, J11 Screw_Terminal_01x02, J12 VAC, J13 NEUTRAL, J14 GND, J17 MCU_GND, J2 GND, J3 MCU_L1, J4 MCU_L2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

Commit message: light board v2
Parts:
- removed J7: MCU_5V, Connector_PinHeader_2.54mm:PinHeader_1x01_P2.54mm_Vertical
- removed Q3: FDD8453LZ, Package_TO_SOT_SMD:TO-252-2
- removed R10, R9: 100k, Resistor_SMD:R_1206_3216Metric
- added J15: 5V, Connector_PinHeader_2.54mm:PinHeader_1x01_P2.54mm_Vertical, F.Cu at (147.0, 125.0)
- added J16: GND, Connector_PinHeader_2.54mm:PinHeader_1x01_P2.54mm_Vertical, F.Cu at (152.0, 125.0)
- added JP1: SolderJumper_2_Open, Jumper:SolderJumper-2_P1.3mm_Open_TrianglePad1.0x1.5mm, F.Cu at (107.0, 95.0)
- added JP2: SolderJumper_2_Open, Jumper:SolderJumper-2_P1.3mm_Open_TrianglePad1.0x1.5mm, F.Cu at (124.0, 95.0)
- added JP3: SolderJumper_2_Open, Jumper:SolderJumper-2_P1.3mm_Open_TrianglePad1.0x1.5mm, F.Cu at (140.0, 95.0)
- added JP4: SolderJumper_2_Open, Jumper:SolderJumper-2_P1.3mm_Open_TrianglePad1.0x1.5mm, F.Cu at (154.0, 119.0)
- D3: value SBR1A20T5-7 -> MBR130HW; footprint Diode_SMD:D_SOD-523 -> Diode_SMD:D_SOD-123
- R1, R2, R3: value 10k -> 150; footprint Resistor_SMD:R_0805_2012Metric -> Resistor_SMD:R_0603_1608Metric
- R5, R7, R8: value 10k -> 1k; footprint Resistor_SMD:R_0805_2012Metric -> Resistor_SMD:R_0603_1608Metric
- moved J1 11.3 mm to (89.0, 96.0)
- moved R2 10.0 mm to (127.0, 110.4)
- moved Q6 9.79 mm to (133.5, 111.1)
- moved R8 9.69 mm to (140.1, 110.5)
- moved R3 9.20 mm to (104.5, 113.1)
- moved Q5 9.19 mm to (111.1, 111.1)
- moved R7 9.19 mm to (118.0, 110.5)
- moved R1 9.10 mm to (104.5, 110.5)
- moved R5 8.86 mm to (117.9, 114.2)
- moved J12 7.74 mm to (167.0, 92.0)
- moved J13 6.19 mm to (167.0, 98.0)
- moved Q1 5.77 mm to (100.5, 98.2)
- moved Q2 5.77 mm to (117.5, 98.2)
- moved Q4 5.77 mm to (133.5, 98.2)
- moved J14 5.29 mm to (89.0, 105.7)
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Connections:
- D3 pad 1: Net-(D3-Pad1) -> MCU_Bike
- J10 pad 1: Net-(J10-Pad1) -> +24V
- J10 pad 2: GND -> Net-(J10-Pad2)
- J11 pad 2: Earth -> VAC
- J8 pad 1: Net-(J8-Pad1) -> +24V
- J8 pad 2: GND -> Net-(J8-Pad2)
- J9 pad 1: Net-(J9-Pad1) -> +24V
- J9 pad 2: GND -> Net-(J9-Pad2)
- K1 pad 1: Net-(D3-Pad1) -> GND1
- K1 pad 3: VAC -> Earth
- K1 pad 6: GND1 -> MCU_Bike
- Q1 pad 2: +24V -> Net-(J8-Pad2)
- Q1 pad 3: Net-(J8-Pad1) -> GND
- Q2 pad 2: +24V -> Net-(J9-Pad2)
- Q2 pad 3: Net-(J9-Pad1) -> GND
- Q4 pad 2: +24V -> Net-(J10-Pad2)
- Q4 pad 3: Net-(J10-Pad1) -> GND
- Q5 pad 6: 12V -> +5V
- Q5 pad 8: 12V -> +5V
- Q6 pad 6: 12V -> +5V
- Q6 pad 8: 12V -> +5V
Routing:
- net 12V: track 56.8 -> 0.00 mm
- net MCU_L2: track 13.1 -> 62.5 mm, vias 0 -> 2
- net +24V: track 6.85 -> 55.3 mm
- net GND1: track 71.1 -> 109.6 mm, vias 6 -> 4
- net +5V: track 21.3 -> 53.8 mm
- net MCU_L1: track 12.2 -> 38.2 mm, vias 2 -> 0
- net Net-(D3-Pad1): track 21.6 -> 0.00 mm
- net MCU_L3: track 17.6 -> 36.3 mm, vias 0 -> 2
- net Net-(J10-Pad2): track 0.00 -> 17.1 mm
- net Net-(J9-Pad2): track 0.00 -> 17.1 mm
- net Net-(J8-Pad2): track 0.00 -> 17.1 mm
- net Earth: track 0.00 -> 15.8 mm
- net MCU_Bike: track 28.1 -> 16.9 mm, vias 2 -> 0
- net Net-(J10-Pad1): track 11.0 -> 0.00 mm
- net Net-(J9-Pad1): track 11.0 -> 0.00 mm
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- removed copper zone on F.Cu, net +24V
- removed copper zone on F.Cu, net Earth
Other:
- board text added: "+24V"
- board text added: "+5V"
- board text added: "BIKE"
- board text added: "GND"
- board text added: "L1"
- board text added: "L2"
- board text added: "L3"
- board text added: "MCU_GND"
- board text added: "NEUTRAL"
- board text added: "Team 20 Light Board v2 3/28/22"
- board text added: "VAC"
- board text removed: "Team 20 Light Board v1 3/6/22"

Commit message: update pcbs
Parts:
- removed J14: GND, Connector_PinHeader_2.54mm:PinHeader_1x01_P2.54mm_Vertical
- J1, J12, J13, J2: footprint Connector_PinHeader_2.54mm:PinHeader_1x01_P2.54mm_Vertical -> _mylib:hole
- moved J17 2.80 mm to (167.0, 109.8)
- moved J13 1.50 mm to (167.1, 99.5)
- moved J1 1.10 mm to (89.0, 94.9)
- moved J2 0.60 mm to (89.0, 101.3)
Routing:
- net GND1: track 109.6 -> 110.9 mm
- net Earth: track 15.8 -> 16.5 mm
- net +24V: track 55.3 -> 54.7 mm
