File: kicad/power_board/power_board.kicad_pcb (KiCad board)
At the start: 2 copper layers, 98.4 x 100 mm, 94 parts, among them IC1 LTC4151IMS-1#PBF, J1 24V, J10 Grid, J11 GRID_CTRL, J12 MCU_2, J14 5V, J15 MCU_P_RES, J16 MCU_BTN1, J17 MCU_BTN2, J18 BTN1, J19 BTN2, J2 24V, J20 MCU_GND, J21 SOLAR_CTRL, J22 CTRL, J3 GND, J4 GND, J5 GND, J6 GND, J7 MCU, J9 Solar Panel, Q1 FDD8453LZ, Q10 MOCD207M, Q2 FDD8453LZ, Q3 FDD8453LZ, Q4 FDD8453LZ, Q5 FDS5670, Q6 MOCD207M, Q7 MOCD207M, Q8 FDD8453LZ, Q9 MOCD207M, U5 LT3757A, U6 LT1161

Commit message: update pcbs
Parts:
- removed C16, C17, C18, C19: 1u, Capacitor_SMD:C_0603_1608Metric
- removed R28, R29: 100k, Resistor_SMD:R_1206_3216Metric
- removed R3, R4, R5, R6: 0, Resistor_SMD:R_2512_6332Metric
- added J13: GND, Connector_PinHeader_2.54mm:PinHeader_1x01_P2.54mm_Vertical, F.Cu at (126.0, 144.8)
- added J23: 24V, _mylib:hole, F.Cu at (179.5, 106.0)
- added J24: GND, _mylib:hole, F.Cu at (179.5, 113.5)
- added J8: 5V_noisy, Connector_PinHeader_2.54mm:PinHeader_1x01_P2.54mm_Vertical, F.Cu at (122.4, 144.8)
- added JP1: SolderJumper_2_Open, Jumper:SolderJumper-2_P1.3mm_Open_TrianglePad1.0x1.5mm, F.Cu at (106.6, 107.0)
- added JP2: SolderJumper_2_Open, Jumper:SolderJumper-2_P1.3mm_Open_TrianglePad1.0x1.5mm, F.Cu at (106.6, 112.0)
- added JP3: SolderJumper_2_Open, Jumper:SolderJumper-2_P1.3mm_Open_TrianglePad1.0x1.5mm, F.Cu at (112.5, 107.0)
- added JP4: SolderJumper_2_Open, Jumper:SolderJumper-2_P1.3mm_Open_TrianglePad1.0x1.5mm, F.Cu at (112.5, 112.0)
- added JP5: SolderJumper_2_Open, Jumper:SolderJumper-2_P1.3mm_Open_TrianglePad1.0x1.5mm, F.Cu at (124.5, 127.1)
- added JP6: SolderJumper_2_Open, Jumper:SolderJumper-2_P1.3mm_Open_TrianglePad1.0x1.5mm, F.Cu at (139.2, 148.2)
- added JP7: SolderJumper_2_Open, Jumper:SolderJumper-2_P1.3mm_Open_TrianglePad1.0x1.5mm, F.Cu at (139.2, 141.3)
- added JP8: SolderJumper_2_Open, Jumper:SolderJumper-2_P1.3mm_Open_TrianglePad1.0x1.5mm, F.Cu at (115.3, 136.3)
- added JP9: SolderJumper_2_Open, Jumper:SolderJumper-2_P1.3mm_Open_TrianglePad1.0x1.5mm, F.Cu at (123.1, 136.3)
- C24, C25: footprint Capacitor_SMD:C_1210_3225Metric -> Capacitor_SMD:C_0805_2012Metric
- J10, J4: footprint Connector_PinHeader_2.54mm:PinHeader_1x01_P2.54mm_Vertical -> _mylib:hole
- J14: value 5V -> MCU_5V
- J6, J9: footprint _mine:73099 -> _mylib:hole_1.6mm
- Q5: footprint Package_TO_SOT_SMD:LFPAK33 -> Package_SO:SOIC-8_3.9x4.9mm_P1.27mm
- R1: footprint Resistor_SMD:R_2512_6332Metric -> Resistor_SMD:R_0603_1608Metric
- R14, R15: value 20k -> 10k
- R16: value 5.1k -> 2.4k
- R17, R20: value 0.51k -> 240; footprint Resistor_SMD:R_0805_2012Metric -> Resistor_SMD:R_0603_1608Metric
- R18, R19: value 10k -> 5.1k; footprint Resistor_SMD:R_0805_2012Metric -> Resistor_SMD:R_0603_1608Metric
- R21: footprint Resistor_THT:R_Axial_DIN0207_L6.3mm_D2.5mm_P10.16mm_Horizontal -> _mylib:TEH140
- R22, R23, R24, R25, R27, R32, R33: value 10k -> 1k; footprint Resistor_SMD:R_0805_2012Metric -> Resistor_SMD:R_0603_1608Metric
- R26, R30, R31: value 10k -> 150; footprint Resistor_SMD:R_0805_2012Metric -> Resistor_SMD:R_0603_1608Metric
- moved J3 53.8 mm to (181.3, 135.4), turned to 90 degrees
- moved J5 47.2 mm to (181.3, 129.0), turned to 90 degrees
- moved C23 46.5 mm to (165.0, 77.0), turned to 0 degrees
- moved C22 41.3 mm to (165.0, 82.0), turned to 0 degrees
- moved R1 25.4 mm to (163.9, 90.3)
- moved C21 25.0 mm to (172.2, 95.0)
- moved C20 22.8 mm to (172.2, 76.0), turned to 0 degrees
- moved D1 22.1 mm to (164.7, 87.4), turned to 0 degrees
- moved R27 10.9 mm to (139.3, 114.3), turned to 0 degrees
- moved J1 7.89 mm to (170.7, 105.4)
- moved J2 7.89 mm to (165.1, 105.4)
- moved J6 6.40 mm to (132.3, 61.9)
- moved J11 6.04 mm to (145.7, 74.2)
- moved J9 4.60 mm to (123.2, 61.9)
- moved J21 4.12 mm to (138.2, 74.2)
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Connections:
- J14 pad 1: +5V -> MCU_5V
- L3 pad 2: Net-(C10-Pad2) -> GND
- L3 pad 3: GND -> Net-(C10-Pad2)
- Q10 pad 6: 12V -> +5V
- Q10 pad 8: 12V -> +5V
- Q6 pad 6: 12V -> +5V
- Q8 pad 2: 24V Solar_2 -> Net-(Q8-Pad2)
- Q8 pad 3: Net-(Q8-Pad3) -> GND
- Q9 pad 6: +5V -> MCU_5V
- Q9 pad 8: +5V -> MCU_5V
- R17 pad 1: +5V -> MCU_5V
- R18 pad 1: +5V -> MCU_5V
- R19 pad 1: +5V -> MCU_5V
- R20 pad 1: +5V -> MCU_5V
- R21 pad 1: Net-(Q8-Pad3) -> 24V Solar_2
- R21 pad 2: GND -> Net-(Q8-Pad2)
- U6 pad 2: Net-(C16-Pad2) -> unconnected-(U6-Pad2)
- U6 pad 4: Net-(C17-Pad2) -> unconnected-(U6-Pad4)
- U6 pad 6: Net-(C18-Pad2) -> unconnected-(U6-Pad6)
- U6 pad 8: Net-(C19-Pad2) -> unconnected-(U6-Pad8)
Routing:
- net MCU_5V: track 0.00 -> 112.5 mm, vias 0 -> 6
- net +5V: track 100.7 -> 49.3 mm, vias 6 -> 4
- net GND1: track 137.3 -> 104.3 mm, vias 0 -> 10
- net 12V: track 21.1 -> 0.00 mm
- net +24V: track 12.8 -> 31.6 mm
- net Net-(J19-Pad1): track 22.6 -> 7.78 mm
- net GND: track 35.2 -> 45.6 mm, vias 31 -> 29
- net ADR1: track 28.5 -> 20.0 mm
- net Net-(J11-Pad1): track 18.9 -> 11.0 mm
- net MCU_P_RES: track 35.9 -> 43.0 mm
- net MCU_SOLAR: track 12.2 -> 18.8 mm, vias 0 -> 2
- net Net-(Q5-Pad1): track 5.64 -> 10.7 mm
- net MCU_GRID: track 9.72 -> 14.7 mm
- net Net-(Q9-Pad3): track 6.31 -> 11.2 mm, vias 0 -> 2
- net Net-(D1-Pad1): track 6.34 -> 2.09 mm
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- added copper zone on F.Cu, net Net-(Q6-Pad5)
- added copper zone on F.Cu, net Net-(Q8-Pad2)
- removed copper zone on F.Cu, net Net-(Q5-Pad1)
- removed copper zone on F.Cu, net Net-(Q8-Pad3)
Other:
- board text added: "+24V"
- board text added: "+5V"
- board text added: "5V"
- board text added: "ADR0"
- board text added: "ADR1"
- board text added: "BTN1"
- board text added: "BTN2"
- board text added: "CTRL"
- board text added: "G S"
- board text added: "GND"
- board text added: "Grid Ctrl"
- board text added: "MCU"
- board text added: "MCU_INPUTS"
- board text added: "Noisy"
- board text added: "P_RES"
- board text added: "SCL"
- board text added: "SDA"
- board text added: "Solar Ctrl"
- board text added: "Team 20 Power Board v2 3/28/22"
- board text removed: "Team 20 Power Board v1 3/6/22"
